Commit message: Add base_footprint

File: src/my_bot/description/robot_core.xacro (robot description, xacro)
@@ -5,4 +5,12 @@
     <!-- BASE LINK -->
     <link name="base_link">
+    </link>
+    <!-- BASE_FOOTPRINT LINK -->
+    <joint name="base_footprint_joint" type="fixed">
+        <parent link="base_link"/>
+        <child link="base_footprint"/>
+        <origin xyz="0 0 0" rpy="0 0 0"/>
+    </joint>
+    <link name="base_footprint">
     </link>
     <!-- CHASSIS LINK -->

Commit message: add mecanum wheels to robbot

File: src/my_bot/description/robot_core.xacro (robot description, xacro)
@@ -3,4 +3,53 @@
     <xacro:include filename="inertial_macros.xacro"/>
     <xacro:include filename="materials.xacro"/>
+    <!-- Define robot constants -->
+    <xacro:property name="base_width"  value="0.145"/>
+    <xacro:property name="base_length" value="0.240"/>
+    <xacro:property name="base_height" value="0.060"/>
+    <xacro:property name="base_mass"   value="1.500"/>
+    <xacro:property name="wheel_radius" value="0.040"/>
+    <xacro:property name="wheel_width"  value="0.035"/>
+    <xacro:property name="wheel_ygap"   value="0.025"/>
+    <xacro:property name="wheel_zoff"   value="0.010"/>
+    <xacro:property name="wheel_xoff"   value="0.085"/>
+    <xacro:property name="wheel_mass"   value="0.100"/>
+    <xacro:property name="imu_width"  value="0.010"/>
+    <xacro:property name="imu_length" value="0.010"/>
+    <xacro:property name="imu_height" value="0.008"/>
+    <xacro:property name="imu_mass"   value="0.010"/>
+    <xacro:property name="lidar_radius" value="0.0375"/>
+    <xacro:property name="lidar_width"  value="0.0380"/>
+    <xacro:property name="lidar_mass"   value="0.2000"/>
+    <xacro:property name="tower_width"  value="0.085"/>
+    <xacro:property name="tower_length" value="0.085"/>
+    <xacro:property name="tower_height" value="0.060"/>
+    <xacro:property name="tower_mass"   value="0.200"/>
+    <xacro:property name="board_1_width"  value="0.060"/>
+    <xacro:property name="board_1_length" value="0.080"/>
+    <xacro:property name="board_1_height" value="0.015"/>
+    <xacro:property name="board_1_mass"   value="0.100"/>
+    <xacro:property name="board_2_width"  value="0.060"/>
+    <xacro:property name="board_2_length" value="0.090"/>
+    <xacro:property name="board_2_height" value="0.025"/>
+    <xacro:property name="board_2_mass"   value="0.200"/>
+    <xacro:property name="antenna_width"  value="0.010"/>
+    <xacro:property name="antenna_length" value="0.040"/>
+    <xacro:property name="antenna_height" value="0.060"/>
+    <xacro:property name="antenna_mass"   value="0.100"/>
+    <!-- Define some commonly used intertial properties  -->
+    <xacro:macro name="box_inertia" params="m w h d">
+        <inertial>
+        <origin xyz="0 0 0" rpy="${pi/2} 0 ${pi/2}"/>
+        <mass value="${m}"/>
+        <inertia ixx="${(m/12) * (h*h + d*d)}" ixy="0.0" ixz="0.0" iyy="${(m/12) * (w*w + d*d)}" iyz="0.0" izz="${(m/12) * (w*w + h*h)}"/>
+        </inertial>
+    </xacro:macro>
+    <xacro:macro name="cylinder_inertia" params="m r h">
+        <inertial>
+        <origin xyz="0 0 0" rpy="${pi/2} 0 0" />
+        <mass value="${m}"/>
+        <inertia ixx="${(m/12) * (3*r*r + h*h)}" ixy = "0" ixz = "0" iyy="${(m/12) * (3*r*r + h*h)}" iyz = "0" izz="${(m/2) * (r*r)}"/>
+        </inertial>
+    </xacro:macro>
     <!-- BASE LINK -->
     <link name="base_link">
@@ -41,107 +90,31 @@
         <material>Gazebo/White</material>
     </gazebo>
-    <!-- REAR LEFT WHEEL LINK -->
-    <joint name="rear_left_wheel_joint" type="continuous">
-        <parent link="base_link"/>
-        <child link="rear_left_wheel"/>
-        <origin xyz="-0.090 0.09675 -0.0375" rpy="-${pi/2} 0 0" />
-        <axis xyz="0 0 1"/>
+<!-- Wheels -->
+  <xacro:macro name="wheel" params="prefix x_reflect y_reflect">
+    <link name="${prefix}_link">
+      <visual>
+        <origin xyz="0 0 0" rpy="0 0 0"/>
+        <geometry>
+            <mesh filename="file:///workspace/src/my_bot/meshes/omni_wheel.dae" scale="0.325 0.325 0.325"/>
+        </geometry>
+      </visual>
+      <collision>
+        <origin xyz="0 0 0" rpy="${pi/2} 0 0"/>
+        <geometry>
+          <cylinder radius="${wheel_radius}" length="${wheel_width}"/>
+        </geometry>
+      </collision>
+      <xacro:cylinder_inertia m="${wheel_mass}" r="${wheel_radius}" h="${wheel_width}"/>
+    </link>
+    <joint name="${prefix}_joint" type="continuous">
+      <parent link="base_link"/>
+      <child  link="${prefix}_link"/>
+      <origin xyz="${x_reflect*wheel_xoff} ${y_reflect*(base_width/2+wheel_ygap)} ${-wheel_zoff}" rpy="0 0 0"/>
+      <axis xyz="0 1 0"/>
     </joint>
-    <link name="rear_left_wheel">
-        <visual>
-            <geometry>
-                <cylinder radius="0.0375" length="0.0325"/>
-            </geometry>
-            <material name="black"/>
-        </visual>
-        <collision>
-            <geometry>
-                <cylinder radius="0.0375" length="0.0325"/>
-            </geometry>
-        </collision>
-        <xacro:inertial_cylinder mass="0.1" length="0.0325" radius="0.0375">
-            <origin xyz="0 0 0" rpy="0 0 0"/>
-        </xacro:inertial_cylinder>
-    </link>
-    <gazebo reference="rear_left_wheel">
-        <material>Gazebo/Black</material>
-    </gazebo>
-    <!-- REAR RIGHT WHEEL LINK -->
-    <joint name="rear_right_wheel_joint" type="continuous">
-        <parent link="base_link"/>
-        <child link="rear_right_wheel"/>
-        <origin xyz="-0.090 -0.09675 -0.0375" rpy="${pi/2} 0 0" />
-        <axis xyz="0 0 -1"/>
-    </joint>
-    <link name="rear_right_wheel">
-        <visual>
-            <geometry>
-                <cylinder radius="0.0375" length="0.0325"/>
-            </geometry>
-            <material name="black"/>
-        </visual>
-        <collision>
-            <geometry>
-                <cylinder radius="0.0375" length="0.0325"/>
-            </geometry>
-        </collision>
-        <xacro:inertial_cylinder mass="0.1" length="0.0325" radius="0.0375">
-            <origin xyz="0 0 0" rpy="0 0 0"/>
-        </xacro:inertial_cylinder>
-    </link>
-    <gazebo reference="rear_right_wheel">
-        <material>Gazebo/Black</material>
-    </gazebo>
-       <!-- FRONT LEFT WHEEL LINK -->
-    <joint name="front_left_wheel_joint" type="continuous">
-        <parent link="base_link"/>
-        <child link="front_left_wheel"/>
-        <origin xyz="0.080 0.09675 -0.0375" rpy="-${pi/2} 0 0" />
-        <axis xyz="0 0 1"/>
-    </joint>
-    <link name="front_left_wheel">
-        <visual>
-            <geometry>
-                <cylinder radius="0.0375" length="0.0325"/>
-            </geometry>
-            <material name="black"/>
-        </visual>
-        <collision>
-            <geometry>
-                <cylinder radius="0.0375" length="0.0325"/>
-            </geometry>
-        </collision>
-        <xacro:inertial_cylinder mass="0.1" length="0.0325" radius="0.0375">
-            <origin xyz="0 0 0" rpy="0 0 0"/>
-        </xacro:inertial_cylinder>
-    </link>
-    <gazebo reference="front_left_wheel">
-        <material>Gazebo/Black</material>
-    </gazebo>
-    <!-- FRONT RIGHT WHEEL LINK -->
-    <joint name="front_right_wheel_joint" type="continuous">
-        <parent link="base_link"/>
-        <child link="front_right_wheel"/>
-        <origin xyz="0.080 -0.09675 -0.0375" rpy="${pi/2} 0 0" />
-        <axis xyz="0 0 -1"/>
-    </joint>
-    <link name="front_right_wheel">
-        <visual>
-            <geometry>
-                <cylinder radius="0.0375" length="0.0325"/>
-            </geometry>
-            <material name="black"/>
-        </visual>
-        <collision>
-            <geometry>
-                <cylinder radius="0.0375" length="0.0325"/>
-            </geometry>
-        </collision>
-        <xacro:inertial_cylinder mass="0.1" length="0.0325" radius="0.0375">
-            <origin xyz="0 0 0" rpy="0 0 0"/>
-        </xacro:inertial_cylinder>
-    </link>
-    <gazebo reference="front_right_wheel">
-        <material>Gazebo/Black</material>
-    </gazebo>
+  </xacro:macro>
+  <xacro:wheel prefix="front_left_wheel"  x_reflect="1"  y_reflect="1"  />
+  <xacro:wheel prefix="front_right_wheel" x_reflect="1"  y_reflect="-1" />
+  <xacro:wheel prefix="rear_left_wheel"   x_reflect="-1" y_reflect="1"  />
+  <xacro:wheel prefix="rear_right_wheel"  x_reflect="-1" y_reflect="-1" />
 </robot>

Commit message: add world to launch_sim

File: src/my_bot/description/robot_core.xacro (robot description, xacro)
@@ -8,5 +8,5 @@
     <xacro:property name="base_height" value="0.060"/>
     <xacro:property name="base_mass"   value="1.500"/>
-    <xacro:property name="wheel_radius" value="0.040"/>
+    <xacro:property name="wheel_radius" value="0.0375"/>
     <xacro:property name="wheel_width"  value="0.035"/>
     <xacro:property name="wheel_ygap"   value="0.025"/>
@@ -21,8 +21,4 @@
     <xacro:property name="lidar_width"  value="0.0380"/>
     <xacro:property name="lidar_mass"   value="0.2000"/>
-    <xacro:property name="tower_width"  value="0.085"/>
-    <xacro:property name="tower_length" value="0.085"/>
-    <xacro:property name="tower_height" value="0.060"/>
-    <xacro:property name="tower_mass"   value="0.200"/>
     <xacro:property name="board_1_width"  value="0.060"/>
     <xacro:property name="board_1_length" value="0.080"/>
@@ -33,8 +29,4 @@
     <xacro:property name="board_2_height" value="0.025"/>
     <xacro:property name="board_2_mass"   value="0.200"/>
-    <xacro:property name="antenna_width"  value="0.010"/>
-    <xacro:property name="antenna_length" value="0.040"/>
-    <xacro:property name="antenna_height" value="0.060"/>
-    <xacro:property name="antenna_mass"   value="0.100"/>
     <!-- Define some commonly used intertial properties  -->
     <xacro:macro name="box_inertia" params="m w h d">
@@ -118,3 +110,92 @@
   <xacro:wheel prefix="rear_left_wheel"   x_reflect="-1" y_reflect="1"  />
   <xacro:wheel prefix="rear_right_wheel"  x_reflect="-1" y_reflect="-1" />
+    <link name="imu_link">
+    <visual>
+      <geometry>
+        <box size="${imu_length} ${imu_width} ${imu_height}"/>
+      </geometry>
+      <material name="Dark Blue">
+        <color rgba="0.0 0.0 0.4 1.0"/>
+      </material>
+    </visual>
+    <collision>
+      <geometry>
+        <box size="${imu_length} ${imu_width} ${imu_height}"/>
+      </geometry>
+    </collision>
+    <xacro:box_inertia m="${imu_mass}" w="${imu_width}" d="${imu_length}" h="${imu_height}"/>
+  </link>
+  <joint name="imu_joint" type="fixed">
+    <parent link="base_link"/>
+    <child  link="imu_link"/>
+    <origin xyz="0.02 -0.02 ${base_height/2 + 0.02}"/>
+  </joint>
+  <gazebo reference="imu_link">
+    <sensor name="imu_sensor" type="imu">
+      <plugin filename="libgazebo_ros_imu_sensor.so" name="imu_plugin">
+        <ros>
+          <namespace>/demo</namespace>
+          <remapping>~/out:=imu</remapping>
+        </ros>
+        <initial_orientation_as_reference>false</initial_orientation_as_reference>
+      </plugin>
+      <always_on>true</always_on>
+      <update_rate>100</update_rate>
+      <visualize>true</visualize>
+     <imu>
+      <angular_velocity>
+        <x>
+          <noise type="gaussian">
+              <mean>0.0</mean>
+              <stddev>2e-4</stddev>
+              <bias_mean>0.0000075</bias_mean>
+              <bias_stddev>0.0000008</bias_stddev>
+            </noise>
+          </x>
+          <y>
+            <noise type="gaussian">
+              <mean>0.0</mean>
+              <stddev>2e-4</stddev>
+              <bias_mean>0.0000075</bias_mean>
+              <bias_stddev>0.0000008</bias_stddev>
+            </noise>
+          </y>
+          <z>
+            <noise type="gaussian">
+              <mean>0.0</mean>
+              <stddev>2e-4</stddev>
+              <bias_mean>0.0000075</bias_mean>
+              <bias_stddev>0.0000008</bias_stddev>
+            </noise>
+          </z>
+        </angular_velocity>
+        <linear_acceleration>
+          <x>
+            <noise type="gaussian">
+              <mean>0.0</mean>
+              <stddev>1.7e-2</stddev>
+              <bias_mean>0.1</bias_mean>
+              <bias_stddev>0.001</bias_stddev>
+            </noise>
+          </x>
+          <y>
+            <noise type="gaussian">
+              <mean>0.0</mean>
+              <stddev>1.7e-2</stddev>
+              <bias_mean>0.1</bias_mean>
+              <bias_stddev>0.001</bias_stddev>
+            </noise>
+          </y>
+          <z>
+            <noise type="gaussian">
+              <mean>0.0</mean>
+              <stddev>1.7e-2</stddev>
+              <bias_mean>0.1</bias_mean>
+              <bias_stddev>0.001</bias_stddev>
+            </noise>
+          </z>
+        </linear_acceleration>
+      </imu>
+    </sensor>
+  </gazebo>
 </robot>
